File: Dreamcast/hw/Dreamdrivecast/_autosave-Dreamdrivecast.kicad_sch (KiCad schematic)
At the start: 3 parts

Commit message: Updating dreamcast schematic with lots of notes about what signals are used for what.
Parts:
- removed U?: Pico, RPi_Pico:RPi_Pico_SMD_TH, symbol MCU_RaspberryPi_and_Boards:Pico
- added U?: WeAct-RP2040-Pico, WeAct-RP2040-Pico:WeAct-RP2040-Pico, symbol Weact-RP2040-Pico:WeAct-RP2040-Pico
Connections:
- net D0: now also U?.1 (GP0)
- net D1: now also U?.2 (GP1)
- net D10: now also U?.14 (GP10)
- net D11: now also U?.15 (GP11)
- net D12: now also U?.16 (GP12)
- net D13: now also U?.17 (GP13)
- net D14: now also U?.19 (GP14)
- net D15: now also U?.20 (GP15)
- net D2: now also U?.4 (GP2)
- net D3: now also U?.5 (GP3)
- net D4: now also U?.6 (GP4)
- net D5: now also U?.7 (GP5)
- net D6: now also U?.9 (GP6)
- net D7: now also U?.10 (GP7)
- net D8: now also U?.11 (GP8)
- net D9: now also U?.12 (GP9)
Other:
- note added: "(audio data, serial)"
- note added: "33.8688 MHz"
- note added: "Bit clock"
- note added: "DMACK- (DMA acknowledge) (optional) This signal is used by the host in response to DMARQ, for initiating a DMA transfer. DMARQ- (DMA request) (optional) This signal is used for DMA transfer between the host and this device. When data transfer is possible, the device drives the signal. The data transfer direction is controlled by the DIOR- and DIOW- commands. This signal is used in handshaking wit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"
- note added: "D[0:15] Bidirectional data bus that can be used either as 8-bit or 16-bit bus."
- note added: "GD-ROM chip selection"
- note added: "IDE_CSO (Chip select 0) Serves for selecting the command block register. Note: This signal is known as "CS1FX-" in the industry. IDE_CS1(Chip select 1) Serves for selecting the control block register. Note: This signal is known as "CS3FX-" in the industry."
- note added: "INTRQ (Device interrupt) Serves for issuing an interrupt to the host. The INTRQ signal has a hold function which asserts the interrupt only when the device is selected and the host has cleared the nIEN bit in the device control register. When the nIEN bit is "1", or when the device is not selected, the INTRQ signal is in the high-impedance state, regardless of the presence of the hold interrupt. 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"
- note added: "IORDY (I/O channel ready) When the device cannot comply with a data transfer request, the signal is negated in order to expand the register access host transfer cycles. When this signal is driven, it is valid only during the DIOR-/DIOW- cycle for the selected device. When the IORDY signal is not negated, it is in the high- impedance state, because it is an open collector signal."
- note added: "Left right clock"
- note added: "RD (Read strobe signal from the host) At the falling edge of this signal, the data on the DDO- DD7, DD8-DD15 data bus from the device register or data port become valid. At the rising edge of this signal, the host latches on to the data. Until latching is completed, the host cannot access the data."
- note added: "RESET (Device reset) This signal is issued by the host. It is asserted at the start of power-on, and the assert state is maintained until the power supply level has stabilized. This is a tolerance interval until device reset after power-on. MCK (Main clock) 33.8688 MHz clock signal for AICA use. BCLK (Bit clock) Clock signal for fetching Digital Audio. LRCK (Left right clock) Digital Audio left/r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"
- note added: "Specifies the register and data read/write port."
- note added: "WR (Write strobe signal from the host) At the falling edge of this signal, the data on DDO- DD7, DD8-DD15 data bus from the device register or data port are latched. Until latching is completed, the device cannot access the data."
- note removed: "(33MHz)"
- note removed: "(audio data)"
- note removed: "CDDA What pins? Some pins are shared between ide and cdda?"
- note removed: "G1 Bus pins not used by GDRom. Used by Flash Memory?"
- moved on the sheet: CN?, JP?
