File: Dreamcast/hw/Dreamdrivecast/Dreamdrivecast.kicad_sch (KiCad schematic)
At the start: 61 parts, among them CN1 Molex_52602_0579, J1 Breakout, J2 POWER, J3 USB_C_Receptacle_USB2.0, J4 USB_C_Receptacle_USB2.0, J5 Micro_SD_Card, SW1 Lid, SW2 MCU1_BOOT, SW3 MCU2_BOOT, U1 TS3L501ERUA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

Commit message: Moved some things around. Wrote a struct to contain all the databus pio programs, should make it easier to swap out the cs detect for read/write detect programs. Still not sure how fast that actually is though. Updated BOM for circuit board as well as added part numbers for all populated parts, so checking that in so my hard work doesn't blow away in the wind. Moved databus pio programs (e.g. cs detect) to "sega_databus" in the "shared" directory. There are a few items that need to be updated but at least this compiles for now.
Parts:
- C1, C13, C14, C15, C16, C17, C18, C19, C2, C20, C21, C24, C3, C4, C5, C6, C7, C8: LCSC (none) -> C1525; MPN (none) -> CL05B104KO5NNNC
- C10, C22, C23, C9: LCSC (none) -> C14445; MPN (none) -> CL05A105KP5NNNC
- C11, C12: LCSC (none) -> C315248; MPN (none) -> CL05A106MP5NUNC
- C25, C26, C27, C28: LCSC (none) -> C106201; MPN (none) -> CC0402JRNPO9BN120
- CN1: LCSC (none) -> C588209
- J3, J4: LCSC (none) -> C2988369; MPN (none) -> GT-USB-7010ASV
- J5: LCSC (none) -> C585350; MPN (none) -> 1040310811
- R10, R2, R3, R9: LCSC (none) -> C284479; MPN (none) -> ARG02FTC27R4
- R11, R12, R4, R5: LCSC (none) -> C25905; MPN (none) -> 0402WGF5101TCE
- R13, R8: LCSC (none) -> C60491; MPN (none) -> RC0402FR-07100KL
- R14, R6: LCSC (none) -> C60490; MPN (none) -> RC0402FR-0710KL
- R15, R7: LCSC (none) -> C25543; MPN (none) -> 0402WGJ0102TCE
- SW2, SW3: LCSC (none) -> C520860; MPN (none) -> TS-1092S-B3D2-G
- U1: LCSC (none) -> C2652454; MPN (none) -> TS3L501ERUAR
- U2, U5: LCSC (none) -> C2040; MPN (none) -> RP2040
- U3: LCSC (none) -> C110474; MPN (none) -> AZ1117H-3.3TRG1
- U4, U6: LCSC (none) -> C97521; MPN (none) -> W25Q128JVSIQ
- Y1, Y2: MPN (none) -> XYDBPCNANF-12MHZ
