File: Dreamcast/hw/Dreamdrivecast-v1b/Dreamdrivecast-v1b/Dreamdrivecast-v1b.kicad_sch (KiCad schematic)
At the start: 12 parts, among them CN1 Molex_52602_0579, J1 USB_C_Receptacle_USB2.0, J2 Micro_SD_Card, J4 Dreamcast Data, J6 Dreamcast Control Lines, J8 Dreamcast Misc, J9 MCU Misc

Commit message: Getting handshake to at least the req_mode command (0x11) but either doesn't like the data or the sector number data is wrong (the disc type and status) or I'm missing something else entirely.
Parts:
- J2: footprint Connector_Card:microSD_HC_Molex_104031-0811 -> sd_card_lib:TF-SMD_TF-PUSH
Changed lines of the file:
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@@
 			)
 		)
-		(property "Footprint" "Connector_Card:microSD_HC_Molex_104031-0811"
+		(property "Footprint" "sd_card_lib:TF-SMD_TF-PUSH"
 			(at 318.77 144.78 0)
 			(effects
